File: kicad/RP2040_KlipperIO/RP2040_KlipperIO.kicad_pcb (KiCad board)
At the start: 2 copper layers, 72 x 50 mm, 1 part

Commit message: Add basic schematic
Parts:
- added C1: 100n, Capacitor_SMD:C_0603_1608Metric_Pad1.08x0.95mm_HandSolder, F.Cu at (-28.1, -43.3)
- added C2: 100n, Capacitor_SMD:C_0603_1608Metric_Pad1.08x0.95mm_HandSolder, F.Cu at (-28.1, -40.8)
- added C3: 100n, Capacitor_SMD:C_0603_1608Metric_Pad1.08x0.95mm_HandSolder, F.Cu at (-28.1, -38.3)
- added C4: 330u, Capacitor_SMD:CP_Elec_10x7.9, F.Cu at (-37.6, -52.9)
- added C5: 330u, Capacitor_SMD:CP_Elec_10x7.9, F.Cu at (-37.6, -41.0)
- added D2: SS34, Diode_SMD:D_SMA_Handsoldering, F.Cu at (-22.2, 1.35)
- added J1: Conn_01x02_Socket, TerminalBlock_RND:TerminalBlock_RND_205-00001_1x02_P5.00mm_Horizontal, F.Cu at (-63.3, -52.8)
- added J10: Conn_01x02_Socket, TerminalBlock_RND:TerminalBlock_RND_205-00001_1x02_P5.00mm_Horizontal, F.Cu at (-63.3, -19.6)
- added J11: Conn_01x03_Pin, Connector_PinHeader_2.54mm:PinHeader_1x03_P2.54mm_Vertical, F.Cu at (-28.8, -20.6)
- added J12: Conn_01x04_Pin, Connector_PinHeader_2.54mm:PinHeader_1x04_P2.54mm_Vertical, F.Cu at (-28.6, -32.8)
- added J13: Conn_01x02_Socket, TerminalBlock_RND:TerminalBlock_RND_205-00001_1x02_P5.00mm_Horizontal, F.Cu at (-63.3, -8.60)
- added J14: Conn_01x03_Pin, Connector_PinHeader_2.54mm:PinHeader_1x03_P2.54mm_Vertical, F.Cu at (-24.2, -20.6)
- added J15: Conn_01x04_Pin, Connector_PinHeader_2.54mm:PinHeader_1x04_P2.54mm_Vertical, F.Cu at (-24.0, -32.8)
- added J16: Conn_01x02_Socket, TerminalBlock_RND:TerminalBlock_RND_205-00001_1x02_P5.00mm_Horizontal, F.Cu at (-63.3, 2.45)
- added J17: Conn_01x04_Pin, TerminalBlock_RND:TerminalBlock_RND_205-00003_1x04_P5.00mm_Horizontal, F.Cu at (15.5, -73.5)
- added J18: Conn_01x04_Pin, TerminalBlock_RND:TerminalBlock_RND_205-00003_1x04_P5.00mm_Horizontal, F.Cu at (36.5, -73.5)
- added J19: Conn_01x04_Pin, TerminalBlock_RND:TerminalBlock_RND_205-00003_1x04_P5.00mm_Horizontal, F.Cu at (-5.50, -73.5)
- added J2: Conn_01x04_Pin, Connector_PinHeader_2.54mm:PinHeader_1x04_P2.54mm_Vertical, F.Cu at (-42.6, -32.8)
- added J20: Conn_01x04_Pin, TerminalBlock_RND:TerminalBlock_RND_205-00003_1x04_P5.00mm_Horizontal, F.Cu at (-5.50, -61.5)
- added J21: Conn_01x04_Pin, TerminalBlock_RND:TerminalBlock_RND_205-00003_1x04_P5.00mm_Horizontal, F.Cu at (15.5, -61.5)
- added J22: Conn_01x04_Pin, TerminalBlock_RND:TerminalBlock_RND_205-00003_1x04_P5.00mm_Horizontal, F.Cu at (36.5, -61.5)
- added J23: Conn_01x06_Pin, TerminalBlock_RND:TerminalBlock_RND_205-00005_1x06_P5.00mm_Horizontal, F.Cu at (59.0, -5.50)
- added J3: Conn_01x03_Pin, Connector_PinHeader_2.54mm:PinHeader_1x03_P2.54mm_Vertical, F.Cu at (-42.6, -20.6)
- added J4: Conn_01x03_Pin, Connector_PinHeader_2.54mm:PinHeader_1x03_P2.54mm_Vertical, F.Cu at (-38.0, -20.6)
- added J5: Conn_01x04_Pin, Connector_PinHeader_2.54mm:PinHeader_1x04_P2.54mm_Vertical, F.Cu at (-38.0, -32.8)
- added J6: Conn_01x02_Socket, TerminalBlock_RND:TerminalBlock_RND_205-00001_1x02_P5.00mm_Horizontal, F.Cu at (-63.3, -41.8)
- added J7: Conn_01x02_Socket, TerminalBlock_RND:TerminalBlock_RND_205-00001_1x02_P5.00mm_Horizontal, F.Cu at (-63.3, -30.7)
- added J8: Conn_01x03_Pin, Connector_PinHeader_2.54mm:PinHeader_1x03_P2.54mm_Vertical, F.Cu at (-33.4, -20.6)
- added J9: Conn_01x04_Pin, Connector_PinHeader_2.54mm:PinHeader_1x04_P2.54mm_Vertical, F.Cu at (-33.3, -32.8)
- added L1: 100u, GioN_Custom:L_12x12mm_H8mm, F.Cu at (-21.6, -51.7)
- added Q1: IRFL4105PBF, Package_TO_SOT_SMD:SOT-223, F.Cu at (-49.9, -54.7)
- added Q2: IRFL4105PBF, Package_TO_SOT_SMD:SOT-223, F.Cu at (-49.9, -46.5)
- added Q3: IRFL4105PBF, Package_TO_SOT_SMD:SOT-223, F.Cu at (-49.9, -38.2)
- added Q4: IRFL4105PBF, Package_TO_SOT_SMD:SOT-223, F.Cu at (-49.9, -29.9)
- added Q5: IRFL4105PBF, Package_TO_SOT_SMD:SOT-223, F.Cu at (-49.9, -21.7)
- added R1: 12k, Resistor_SMD:R_0201_0603Metric_Pad0.64x0.40mm_HandSolder, F.Cu at (-25.8, -12.3)
- added R10: 2k7, Resistor_SMD:R_0201_0603Metric_Pad0.64x0.40mm_HandSolder, F.Cu at (-23.0, -8.80)
- added R11: 5k1, Resistor_SMD:R_0201_0603Metric_Pad0.64x0.40mm_HandSolder, F.Cu at (-23.0, -7.05)
- added R12: 100R, Resistor_SMD:R_0201_0603Metric_Pad0.64x0.40mm_HandSolder, F.Cu at (-23.0, -5.30)
- added R13: 2k7, Resistor_SMD:R_0201_0603Metric_Pad0.64x0.40mm_HandSolder, F.Cu at (-23.0, -3.55)
- added R14: 5k1, Resistor_SMD:R_0201_0603Metric_Pad0.64x0.40mm_HandSolder, F.Cu at (-23.0, -1.80)
- added R15: 100R, Resistor_SMD:R_0201_0603Metric_Pad0.64x0.40mm_HandSolder, F.Cu at (-20.2, -12.3)
- added R16: 2k7, Resistor_SMD:R_0201_0603Metric_Pad0.64x0.40mm_HandSolder, F.Cu at (-20.2, -10.6)
- added R17: 5k1, Resistor_SMD:R_0201_0603Metric_Pad0.64x0.40mm_HandSolder, F.Cu at (-20.2, -8.80)
- added R18: 100R, Resistor_SMD:R_0201_0603Metric_Pad0.64x0.40mm_HandSolder, F.Cu at (-20.2, -7.05)
- added R2: 1k5, Resistor_SMD:R_0201_0603Metric_Pad0.64x0.40mm_HandSolder, F.Cu at (-25.8, -10.6)
- added R3: 1k, Resistor_SMD:R_0201_0603Metric_Pad0.64x0.40mm_HandSolder, F.Cu at (-25.8, -8.80)
- added R4: 2k7, Resistor_SMD:R_0201_0603Metric_Pad0.64x0.40mm_HandSolder, F.Cu at (-25.8, -7.05)
- added R5: 5k1, Resistor_SMD:R_0201_0603Metric_Pad0.64x0.40mm_HandSolder, F.Cu at (-25.8, -5.30)
- added R6: 2k7, Resistor_SMD:R_0201_0603Metric_Pad0.64x0.40mm_HandSolder, F.Cu at (-25.8, -3.55)
- added R7: 5k1, Resistor_SMD:R_0201_0603Metric_Pad0.64x0.40mm_HandSolder, F.Cu at (-25.8, -1.80)
- added R8: 100R, Resistor_SMD:R_0201_0603Metric_Pad0.64x0.40mm_HandSolder, F.Cu at (-23.0, -12.3)
- added R9: 100R, Resistor_SMD:R_0201_0603Metric_Pad0.64x0.40mm_HandSolder, F.Cu at (-23.0, -10.6)
- added U1: 74HC14, Package_SO:SOIC-14_3.9x8.7mm_P1.27mm, F.Cu at (-17.4, -30.0)
- added U2: LM2576HVS-ADJ, Package_TO_SOT_SMD:TO-263-5_TabPin3, F.Cu at (-34.2, -7.00)
Connections:
- D1 pad 1: unconnected-(D1-GPIO0-Pad1) -> Net-(D1-GPIO0)
- D1 pad 10: unconnected-(D1-GPIO7-Pad10) -> SENSE_FAN3
- D1 pad 11: unconnected-(D1-GPIO8-Pad11) -> PWM_FAN4
- D1 pad 12: unconnected-(D1-GPIO9-Pad12) -> SENSE_FAN4
- D1 pad 14: unconnected-(D1-GPIO10-Pad14) -> ENABLE_STEPPER
- D1 pad 15: unconnected-(D1-GPIO11-Pad15) -> DIR_0
- D1 pad 16: unconnected-(D1-GPIO12-Pad16) -> STEP_0
- D1 pad 17: unconnected-(D1-GPIO13-Pad17) -> DIR_1
- D1 pad 19: unconnected-(D1-GPIO14-Pad19) -> STEP_1
- D1 pad 2: unconnected-(D1-GPIO1-Pad2) -> Net-(D1-GPIO1)
- D1 pad 20: unconnected-(D1-GPIO15-Pad20) -> DIR_2
- D1 pad 21: unconnected-(D1-GPIO16-Pad21) -> STEP_2
- D1 pad 22: unconnected-(D1-GPIO17-Pad22) -> DIR_3
- D1 pad 24: unconnected-(D1-GPIO18-Pad24) -> STEP_3
- D1 pad 25: unconnected-(D1-GPIO19-Pad25) -> DIR_4
- D1 pad 26: unconnected-(D1-GPIO20-Pad26) -> STEP_4
- D1 pad 27: unconnected-(D1-GPIO21-Pad27) -> DIR_5
- D1 pad 29: unconnected-(D1-GPIO22-Pad29) -> STEP_5
- D1 pad 31: unconnected-(D1-GPIO26-Pad31) -> Net-(D1-GPIO26)
- D1 pad 32: unconnected-(D1-GPIO27-Pad32) -> Net-(D1-GPIO27)
- D1 pad 34: unconnected-(D1-GPIO28-Pad34) -> Net-(D1-GPIO28)
- D1 pad 35: unconnected-(D1-GPIO29-Pad35) -> Net-(D1-GPIO29)
- D1 pad 37: unconnected-(D1-GPIO23-Pad37) -> Net-(D1-GPIO23)
- D1 pad 4: unconnected-(D1-GPIO2-Pad4) -> Net-(D1-GPIO2)
- D1 pad 5: unconnected-(D1-GPIO3-Pad5) -> Net-(D1-GPIO3)
- D1 pad 6: unconnected-(D1-GPIO4-Pad6) -> Net-(D1-GPIO4)
- D1 pad 7: unconnected-(D1-GPIO5-Pad7) -> Net-(D1-GPIO5)
- D1 pad 9: unconnected-(D1-GPIO6-Pad9) -> PWM_FAN3

Commit message: route pcb
Parts:
- J12, J15, J2, J5, J9: footprint Connector_PinHeader_2.54mm:PinHeader_1x04_P2.54mm_Vertical -> Connector_Molex:Molex_KK-254_AE-6410-04A_1x04_P2.54mm_Vertical
- R1, R10, R11, R12, R13, R14, R15, R16, R17, R18, R2, R3, R4, R5, R6, R7, R8, R9: footprint Resistor_SMD:R_0201_0603Metric_Pad0.64x0.40mm_HandSolder -> Resistor_SMD:R_0603_1608Metric_Pad0.98x0.95mm_HandSolder
- moved J16 153.3 mm to (55.0, -95.0)
- moved J13 142.0 mm to (66.6, -66.0), turned to -90 degrees
- moved J6 132.3 mm to (66.6, -16.2), turned to -90 degrees
- moved J10 131.2 mm to (66.6, -38.6), turned to -90 degrees
- moved J7 129.9 mm to (66.6, -27.4), turned to -90 degrees
- moved J1 129.7 mm to (57.9, -6.60), turned to 180 degrees
- moved Q5 124.5 mm to (57.4, -84.8), turned to 90 degrees
- moved Q4 118.7 mm to (66.5, -53.3)
- moved Q1 109.4 mm to (56.4, -28.4)
- moved R18 106.8 mm to (51.9, -85.9)
- moved Q2 106.7 mm to (56.4, -36.1)
- moved Q3 106.4 mm to (56.4, -43.7)
- moved J8 102.9 mm to (55.9, -71.6), turned to 180 degrees
- moved R13 102.3 mm to (56.0, -68.6)
- moved R16 101.8 mm to (48.3, -85.9), turned to 180 degrees
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Routing:
- net ENABLE_STEPPER: track 0.00 -> 208.0 mm
- net +12V: track 0.00 -> 174.1 mm, vias 0 -> 2
- net +24V: track 0.00 -> 174.1 mm, vias 0 -> 2
- net Net-(J12-Pin_4): track 0.00 -> 98.1 mm, vias 0 -> 5
- net Net-(J9-Pin_4): track 0.00 -> 81.5 mm, vias 0 -> 4
- net Net-(J5-Pin_4): track 0.00 -> 69.1 mm, vias 0 -> 4
- net Net-(J2-Pin_4): track 0.00 -> 61.8 mm, vias 0 -> 3
- net Net-(J15-Pin_4): track 0.00 -> 57.3 mm, vias 0 -> 6
- net Net-(D1-GPIO29): track 0.00 -> 57.0 mm
- net Net-(D1-GPIO23): track 0.00 -> 55.9 mm
- net Net-(D1-GPIO26): track 0.00 -> 55.8 mm
- net Net-(D1-GPIO27): track 0.00 -> 55.3 mm
- net Net-(J10-Pin_1): track 0.00 -> 53.4 mm, vias 0 -> 1
- net Net-(D1-GPIO28): track 0.00 -> 53.1 mm
- net Net-(J2-Pin_2): track 0.00 -> 52.7 mm
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- added copper zone on B.Cu, net GND
- added copper zone on F.Cu, net GND
Other:
- board size 72 x 50 mm -> 72 x 100 mm
