File: kicad/RP2040_KlipperIO/RP2040_KlipperIO.kicad_sch (KiCad schematic)
At the start: 1 part

Commit message: Add basic schematic
Parts:
- added C1, C2, C3: 100n, Capacitor_SMD:C_0603_1608Metric_Pad1.08x0.95mm_HandSolder, symbol Device:C
- added C4, C5: 330u, Capacitor_SMD:CP_Elec_10x7.9, symbol Device:C_Polarized
- added D2: SS34, Diode_SMD:D_SMA_Handsoldering, symbol Device:D_Schottky
- added J1, J10, J13, J16, J6, J7: Conn_01x02_Socket, TerminalBlock_RND:TerminalBlock_RND_205-00001_1x02_P5.00mm_Horizontal, symbol Connector:Conn_01x02_Socket
- added J11, J14, J3, J4, J8: Conn_01x03_Pin, Connector_PinHeader_2.54mm:PinHeader_1x03_P2.54mm_Vertical, symbol Connector:Conn_01x03_Pin
- added J12, J15, J2, J5, J9: Conn_01x04_Pin, Connector_PinHeader_2.54mm:PinHeader_1x04_P2.54mm_Vertical, symbol Connector:Conn_01x04_Pin
- added J17, J18, J19, J20, J21, J22: Conn_01x04_Pin, TerminalBlock_RND:TerminalBlock_RND_205-00003_1x04_P5.00mm_Horizontal, symbol Connector:Conn_01x04_Pin
- added J23: Conn_01x06_Pin, TerminalBlock_RND:TerminalBlock_RND_205-00005_1x06_P5.00mm_Horizontal, symbol Connector:Conn_01x06_Pin
- added L1: 100u, GioN_Custom:L_12x12mm_H8mm, symbol Device:L
- added Q1, Q2, Q3, Q4, Q5: IRFL4105PBF, Package_TO_SOT_SMD:SOT-223, symbol Transistor_FET:IRF540N
- added R1: 12k, Resistor_SMD:R_0201_0603Metric_Pad0.64x0.40mm_HandSolder, symbol Device:R
- added R10, R13, R16, R4, R6: 2k7, Resistor_SMD:R_0201_0603Metric_Pad0.64x0.40mm_HandSolder, symbol Device:R
- added R11, R14, R17, R5, R7: 5k1, Resistor_SMD:R_0201_0603Metric_Pad0.64x0.40mm_HandSolder, symbol Device:R
- added R12, R15, R18, R8, R9: 100R, Resistor_SMD:R_0201_0603Metric_Pad0.64x0.40mm_HandSolder, symbol Device:R
- added R2: 1k5, Resistor_SMD:R_0201_0603Metric_Pad0.64x0.40mm_HandSolder, symbol Device:R
- added R3: 1k, Resistor_SMD:R_0201_0603Metric_Pad0.64x0.40mm_HandSolder, symbol Device:R
- added U1: 74HC14, Package_SO:SOIC-14_3.9x8.7mm_P1.27mm, symbol 74xx:74HC14
- added U2: LM2576HVS-ADJ, Package_TO_SOT_SMD:TO-263-5_TabPin3, symbol Regulator_Switching:LM2576HVS-ADJ
Connections:
- net +5V: now also C1.1, U1.14 (VCC)
- net GND: now also C1.2, C2.2, C3.2, C4.2, C5.2, D2.2 (A), J1.2 (Pin_2), J12.1 (Pin_1), J15.1 (Pin_1), J17.1 (Pin_1), J18.1 (Pin_1), J19.1 (Pin_1), J2.1 (Pin_1), J20.1 (Pin_1), J21.1 (Pin_1), J22.1 (Pin_1), J23.1 (Pin_1), J5.1 (Pin_1), J9.1 (Pin_1), Q1.3 (S), Q2.3 (S), Q3.3 (S), Q4.3 (S), Q5.3 (S), R11.2, R14.2, R17.2, R2.1, R5.2, R7.2, U1.13, U1.7 (GND), U2.3 (GND), U2.5 (~{ON}/OFF)
- net at D1.1 (GPIO0): now also U1.1
- net SENSE_FAN3: now reaches D1.10 (GPIO7)
- net SENSE_FAN3: now also R13.2, R14.1
- net PWM_FAN4: now reaches D1.11 (GPIO8)
- net PWM_FAN4: now also U1.11
- net SENSE_FAN4: now reaches D1.12 (GPIO9)
- net SENSE_FAN4: now also R16.2, R17.1
- net ENABLE_STEPPER: now reaches D1.14 (GPIO10)
- net ENABLE_STEPPER: now also J17.2 (Pin_2), J18.2 (Pin_2), J19.2 (Pin_2), J20.2 (Pin_2), J21.2 (Pin_2), J22.2 (Pin_2)
- net DIR_0: now reaches D1.15 (GPIO11)
- net DIR_0: now also J18.4 (Pin_4)
- net STEP_0: now reaches D1.16 (GPIO12)
- net STEP_0: now also J18.3 (Pin_3)
- net DIR_1: now reaches D1.17 (GPIO13)
- net DIR_1: now also J17.4 (Pin_4)
- net STEP_1: now reaches D1.19 (GPIO14)
- net STEP_1: now also J17.3 (Pin_3)
- net at D1.2 (GPIO1): now also R4.2, R5.1
- net DIR_2: now reaches D1.20 (GPIO15)
- net DIR_2: now also J19.4 (Pin_4)
- net STEP_2: now reaches D1.21 (GPIO16)
- net STEP_2: now also J19.3 (Pin_3)
- net DIR_3: now reaches D1.22 (GPIO17)
- net DIR_3: now also J20.4 (Pin_4)
- net STEP_3: now reaches D1.24 (GPIO18)
- net STEP_3: now also J20.3 (Pin_3)
- net DIR_4: now reaches D1.25 (GPIO19)
- net DIR_4: now also J21.4 (Pin_4)
- net STEP_4: now reaches D1.26 (GPIO20)
- net STEP_4: now also J21.3 (Pin_3)
- net DIR_5: now reaches D1.27 (GPIO21)
- net DIR_5: now also J22.4 (Pin_4)
- net STEP_5: now reaches D1.29 (GPIO22)
- net STEP_5: now also J22.3 (Pin_3)
- net at D1.32 (GPIO27): now also J23.5 (Pin_5)
- net at D1.34 (GPIO28): now also J23.4 (Pin_4)
- net at D1.35 (GPIO29): now also J23.3 (Pin_3)
- net at D1.37 (GPIO23): now also J23.2 (Pin_2)
- net at D1.4 (GPIO2): now also U1.3
- net at D1.5 (GPIO3): now also R6.2, R7.1
- net at D1.6 (GPIO4): now also U1.5
- net at D1.7 (GPIO5): now also R10.2, R11.1
- net PWM_FAN3: now reaches D1.9 (GPIO6)
- net PWM_FAN3: now also U1.9
- new net: J15.3 (Pin_3), R16.1
- new net: Q3.1 (G), R12.2
- new net: J10.2 (Pin_2), Q3.2 (D)
- new net: J5.4 (Pin_4), R9.1, U1.4
- new net: J15.4 (Pin_4), R18.1, U1.10
- new net: J9.4 (Pin_4), R12.1, U1.6
- new net: D1.31 (Run), J23.6 (Pin_6)
- new net: Q1.1 (G), R8.2
- new net: J6.2 (Pin_2), Q1.2 (D)
- new net: J4.2 (Pin_2), J5.2 (Pin_2), J7.1 (Pin_1)
- new net: J7.2 (Pin_2), Q2.2 (D)
- new net: J14.2 (Pin_2), J15.2 (Pin_2), J16.1 (Pin_1)
- new net: J10.1 (Pin_1), J8.2 (Pin_2), J9.2 (Pin_2)
- new net: J5.3 (Pin_3), R6.1
- new net: Q2.1 (G), R9.2
- new net: J9.3 (Pin_3), R10.1
- new net: J2.4 (Pin_4), R8.1, U1.2
- new net: Q5.1 (G), R18.2
- new net: J16.2 (Pin_2), Q5.2 (D)
- new net: R2.2, R3.2, U2.4 (FB)
- new net: J11.2 (Pin_2), J12.2 (Pin_2), J13.1 (Pin_1)
- new net: J13.2 (Pin_2), Q4.2 (D)
- new net: J2.3 (Pin_3), R4.1
- new net: J12.4 (Pin_4), R15.1, U1.8
- new net: Q4.1 (G), R15.2
- new net: J2.2 (Pin_2), J3.2 (Pin_2), J6.1 (Pin_1)
- new net: J12.3 (Pin_3), R13.1
- new net: R1.2, R3.1
- new net: D2.1 (K), L1.1, U2.2 (OUT)
- new net +12V: C3.1, C5.1, J11.1 (Pin_1), J14.1 (Pin_1), J3.1 (Pin_1), J4.1 (Pin_1), J8.1 (Pin_1), L1.2, R1.1
- new net +24V: C2.1, C4.1, J1.1 (Pin_1), J11.3 (Pin_3), J14.3 (Pin_3), J3.3 (Pin_3), J4.3 (Pin_3), J8.3 (Pin_3), U2.1 (VIN)

Commit message: route pcb
Parts:
- J12, J15, J2, J5, J9: footprint Connector_PinHeader_2.54mm:PinHeader_1x04_P2.54mm_Vertical -> Connector_Molex:Molex_KK-254_AE-6410-04A_1x04_P2.54mm_Vertical
- R1, R10, R11, R12, R13, R14, R15, R16, R17, R18, R2, R3, R4, R5, R6, R7, R8, R9: footprint Resistor_SMD:R_0201_0603Metric_Pad0.64x0.40mm_HandSolder -> Resistor_SMD:R_0603_1608Metric_Pad0.98x0.95mm_HandSolder
Changed lines of the file:
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@@
       (effects (font (size 1.27 1.27)) (justify left))
     )
-    (property "Footprint" "Resistor_SMD:R_0201_0603Metric_Pad0.64x0.40mm_HandSolder" (at 193.802 130.81 90)
+    (property "Footprint" "Resistor_SMD:R_0603_1608Metric_Pad0.98x0.95mm_HandSolder" (at 193.802 130.81 90)
       (effects (font (size 1.27 1.27)) hide)
     )
@@
       (effects (font (size 1.27 1.27)) (justify left))
     )
-    (property "Footprint" "Resistor_SMD:R_0201_0603Metric_Pad0.64x0.40mm_HandSolder" (at 93.472 106.68 90)
+    (property "Footprint" "Resistor_SMD:R_0603_1608Metric_Pad0.98x0.95mm_HandSolder" (at 93.472 106.68 90)
       (effects (font (size 1.27 1.27)) hide)
     )
@@
       (effects (font (size 1.27 1.27)))
     )
-    (property "Footprint" "Resistor_SMD:R_0201_0603Metric_Pad0.64x0.40mm_HandSolder" (at 123.19 138.938 90)
+    (property "Footprint" "Resistor_SMD:R_0603_1608Metric_Pad0.98x0.95mm_HandSolder" (at 123.19 138.938 90)
       (effects (font (size 1.27 1.27)) hide)
     )
@@
       (effects (font (size 1.27 1.27)) (justify left))
     )
-    (property "Footprint" "Resistor_SMD:R_0201_0603Metric_Pad0.64x0.40mm_HandSolder" (at 193.802 90.17 90)
+    (property "Footprint" "Resistor_SMD:R_0603_1608Metric_Pad0.98x0.95mm_HandSolder" (at 193.802 90.17 90)
       (effects (font (size 1.27 1.27)) hide)
     )
@@
       (effects (font (size 1.27 1.27)) (justify right))
     )
-    (property "Footprint" "Connector_PinHeader_2.54mm:PinHeader_1x04_P2.54mm_Vertical" (at 110.49 93.98 0)
+    (property "Footprint" "Connector_Molex:Molex_KK-254_AE-6410-04A_1x04_P2.54mm_Vertical" (at 110.49 93.98 0)
       (effects (font (size 1.27 1.27)) hide)
     )
@@
       (effects (font (size 1.27 1.27)))
     )
-    (property "Footprint" "Resistor_SMD:R_0201_0603Metric_Pad0.64x0.40mm_HandSolder" (at 123.19 88.138 90)
+    (property "Footprint" "Resistor_SMD:R_0603_1608Metric_Pad0.98x0.95mm_HandSolder" (at 123.19 88.138 90)
       (effects (font (size 1.27 1.27)) hide)
     )
@@
       (effects (font (size 1.27 1.27)) (justify left))
     )
-    (property "Footprint" "Resistor_SMD:R_0201_0603Metric_Pad0.64x0.40mm_HandSolder" (at 93.472 147.32 90)
+    (property "Footprint" "Resistor_SMD:R_0603_1608Metric_Pad0.98x0.95mm_HandSolder" (at 93.472 147.32 90)
       (effects (font (size 1.27 1.27)) hide)
     )
@@
       (effects (font (size 1.27 1.27)) (justify left))
     )
-    (property "Footprint" "Resistor_SMD:R_0201_0603Metric_Pad0.64x0.40mm_HandSolder" (at 93.472 96.52 90)
+    (property "Footprint" "Resistor_SMD:R_0603_1608Metric_Pad0.98x0.95mm_HandSolder" (at 93.472 96.52 90)
       (effects (font (size 1.27 1.27)) hide)
     )
@@
       (effects (font (size 1.27 1.27)))
     )
-    (property "Footprint" "Resistor_SMD:R_0201_0603Metric_Pad0.64x0.40mm_HandSolder" (at 123.19 37.338 90)
+    (property "Footprint" "Resistor_SMD:R_0603_1608Metric_Pad0.98x0.95mm_HandSolder" (at 123.19 37.338 90)
       (effects (font (size 1.27 1.27)) hide)
     )
@@
       (effects (font (size 1.27 1.27)))
     )
-    (property "Footprint" "Resistor_SMD:R_0201_0603Metric_Pad0.64x0.40mm_HandSolder" (at 251.46 50.038 90)
+    (property "Footprint" "Resistor_SMD:R_0603_1608Metric_Pad0.98x0.95mm_HandSolder" (at 251.46 50.038 90)
       (effects (font (size 1.27 1.27)) hide)
     )
@@
       (effects (font (size 1.27 1.27)) (justify left))
     )
-    (property "Footprint" "Resistor_SMD:R_0201_0603Metric_Pad0.64x0.40mm_HandSolder" (at 93.472 55.88 90)
+    (property "Footprint" "Resistor_SMD:R_0603_1608Metric_Pad0.98x0.95mm_HandSolder" (at 93.472 55.88 90)
       (effects (font (size 1.27 1.27)) hide)
     )
@@
       (effects (font (size 1.27 1.27)) (justify left))
     )
-    (property "Footprint" "Resistor_SMD:R_0201_0603Metric_Pad0.64x0.40mm_HandSolder" (at 93.472 45.72 90)
+    (property "Footprint" "Resistor_SMD:R_0603_1608Metric_Pad0.98x0.95mm_HandSolder" (at 93.472 45.72 90)
       (effects (font (size 1.27 1.27)) hide)
     )
@@
       (effects (font (size 1.27 1.27)))
     )
-    (property "Footprint" "Resistor_SMD:R_0201_0603Metric_Pad0.64x0.40mm_HandSolder" (at 223.52 71.628 90)
+    (property "Footprint" "Resistor_SMD:R_0603_1608Metric_Pad0.98x0.95mm_HandSolder" (at 223.52 71.628 90)
       (effects (font (size 1.27 1.27)) hide)
     )
@@
       (effects (font (size 1.27 1.27)) (justify right))
     )
-    (property "Footprint" "Connector_PinHeader_2.54mm:PinHeader_1x04_P2.54mm_Vertical" (at 110.49 144.78 0)
+    (property "Footprint" "Connector_Molex:Molex_KK-254_AE-6410-04A_1x04_P2.54mm_Vertical" (at 110.49 144.78 0)
       (effects (font (size 1.27 1.27)) hide)
     )
@@
       (effects (font (size 1.27 1.27)) (justify right))
     )
-    (property "Footprint" "Connector_PinHeader_2.54mm:PinHeader_1x04_P2.54mm_Vertical" (at 210.82 77.47 0)
+    (property "Footprint" "Connector_Molex:Molex_KK-254_AE-6410-04A_1x04_P2.54mm_Vertical" (at 210.82 77.47 0)
       (effects (font (size 1.27 1.27)) hide)
     )
@@
       (effects (font (size 1.27 1.27)) (justify right))
     )
-    (property "Footprint" "Connector_PinHeader_2.54mm:PinHeader_1x04_P2.54mm_Vertical" (at 110.49 43.18 0)
+    (property "Footprint" "Connector_Molex:Molex_KK-254_AE-6410-04A_1x04_P2.54mm_Vertical" (at 110.49 43.18 0)
       (effects (font (size 1.27 1.27)) hide)
     )
@@
       (effects (font (size 1.27 1.27)) (justify left))
     )
-    (property "Footprint" "Resistor_SMD:R_0201_0603Metric_Pad0.64x0.40mm_HandSolder" (at 259.842 41.91 90)
+    (property "Footprint" "Resistor_SMD:R_0603_1608Metric_Pad0.98x0.95mm_HandSolder" (at 259.842 41.91 90)
       (effects (font (size 1.27 1.27)) hide)
     )
@@
       (effects (font (size 1.27 1.27)) (justify left))
     )
-    (property "Footprint" "Resistor_SMD:R_0201_0603Metric_Pad0.64x0.40mm_HandSolder" (at 93.472 157.48 90)
+    (property "Footprint" "Resistor_SMD:R_0603_1608Metric_Pad0.98x0.95mm_HandSolder" (at 93.472 157.48 90)
       (effects (font (size 1.27 1.27)) hide)
     )
@@
       (effects (font (size 1.27 1.27)))
     )
-    (property "Footprint" "Resistor_SMD:R_0201_0603Metric_Pad0.64x0.40mm_HandSolder" (at 223.52 122.428 90)
+    (property "Footprint" "Resistor_SMD:R_0603_1608Metric_Pad0.98x0.95mm_HandSolder" (at 223.52 122.428 90)
       (effects (font (size 1.27 1.27)) hide)
     )
@@
       (effects (font (size 1.27 1.27)) (justify left))
     )
-    (property "Footprint" "Resistor_SMD:R_0201_0603Metric_Pad0.64x0.40mm_HandSolder" (at 259.842 33.02 90)
+    (property "Footprint" "Resistor_SMD:R_0603_1608Metric_Pad0.98x0.95mm_HandSolder" (at 259.842 33.02 90)
       (effects (font (size 1.27 1.27)) hide)
     )
@@
       (effects (font (size 1.27 1.27)) (justify right))
     )
-    (property "Footprint" "Connector_PinHeader_2.54mm:PinHeader_1x04_P2.54mm_Vertical" (at 210.82 128.27 0)
+    (property "Footprint" "Connector_Molex:Molex_KK-254_AE-6410-04A_1x04_P2.54mm_Vertical" (at 210.82 128.27 0)
       (effects (font (size 1.27 1.27)) hide)
     )
@@
       (effects (font (size 1.27 1.27)) (justify left))
     )
-    (property "Footprint" "Resistor_SMD:R_0201_0603Metric_Pad0.64x0.40mm_HandSolder" (at 193.802 80.01 90)
+    (property "Footprint" "Resistor_SMD:R_0603_1608Metric_Pad0.98x0.95mm_HandSolder" (at 193.802 80.01 90)
       (effects (font (size 1.27 1.27)) hide)
     )
@@
       (effects (font (size 1.27 1.27)) (justify left))
     )
-    (property "Footprint" "Resistor_SMD:R_0201_0603Metric_Pad0.64x0.40mm_HandSolder" (at 193.802 140.97 90)
-      (effects (font (size 1.27 1.27)) hide)
-    )
+    (property "Footprint" "Resistor_SMD:R_0603_1608Metric_Pad0.98x0.95mm_HandSolder" (at 193.802 140.97 90)
+      (effects (font (size 1.27 1.27)) hide)
+    )
